Commit message: Rename Package

File: urdf/URDF.urdf (robot description, URDF)
Before this commit: robot URDF, 6 links, 5 joints
Links:
- link base_Link: geometry collision mesh filename=package://robotic_arm_control/meshes/base_Link.STL; visual mesh filename=package://robotic_arm_control/meshes/base_Link.STL
- link link1_Link: geometry collision mesh filename=package://robotic_arm_control/meshes/link1_Link.STL; visual mesh filename=package://robotic_arm_control/meshes/link1_Link.STL
- link link2_Link: geometry collision mesh filename=package://robotic_arm_control/meshes/link2_Link.STL; visual mesh filename=package://robotic_arm_control/meshes/link2_Link.STL
- link rover_link: geometry collision mesh filename=package://robotic_arm_control/meshes/rover_link.STL; visual mesh filename=package://robotic_arm_control/meshes/rover_link.STL
